Commit message: modified xacrofile to add gps

File: erp42_vehicle/erp42_vehicle_description/urdf/erp42_vehicle.urdf.xacro (robot description, xacro)
@@ -18,8 +18,8 @@
   <!-- Include xacro for inertials, materials and wheels -->
   <xacro:include filename="$(find erp42_vehicle_description)/urdf/wheel.xacro" />
+  <xacro:include filename="$(find erp42_vehicle_description)/urdf/gps_sensor.xacro" />
   <xacro:include filename="$(find velodyne_description)/urdf/VLP-16.urdf.xacro" />
   <xacro:property name="robot_namespace" value="/erp42_vehicle" />
   <!-- Gazebo plugins -->
-  <!-- chson commented230313 -->
   <gazebo>
     <!-- Load ros_control plugin using the steer_bot_hardware_gazebo
@@ -54,25 +54,4 @@
   <xacro:property name="axle_offset" value="0.225" />
   <xacro:property name="steer_offset" value="0.1" />
-  <!-- Base link -->
-  <!-- <link name="dummy">
-   </link> -->
-  <!-- <link name="base_imu" />
-<joint name="base_imu_joint" type="fixed">
-  <parent link="base_footprint" />
-  <child link="base_link" />
-</joint> -->
-<!-- <link name="map">
-</link>
-  <joint name="map_odom_joint" type="fixed">
-    <parent link="map" />
-    <child link="odom" />
-  </joint>
-  <link name="odom">
-    <origin xyz="0 0 0" rpy="0 0 0" />
-  </link>
-  <joint name="odom_base_joint" type="floating">
-    <parent link="odom" />
-    <child link="base_link" />
-  </joint> -->
   <link name="base_link">
     <origin xyz="0 0 0" rpy="0 0 0" />
@@ -97,4 +76,7 @@
       x="${base_length}" y="${base_width}" z="${base_height}" />
   </link>
+    <xacro:gps_sensor namespace="" parent_link="base_link">
+      <origin xyz="0 0 1" rpy="0 0 0" />
+  </xacro:gps_sensor>
   <!-- Front steer and rear wheel joints required for ackermann_steering_controller -->
   <xacro:front_steer
@@ -194,29 +176,4 @@
     </visual>
   </link>
-  <link name="gps_link">
-    <visual>
-      <geometry>
-        <box size="0.1 0.1 0.025" />
-      </geometry>
-      <material name="white">
-        <color rgba="1 1 1 1" />
-      </material>
-    </visual>
-    <collision>
-      <geometry>
-        <sphere radius="0.05" />
-      </geometry>
-    </collision>
-    <inertial>
-      <mass value="0.1" />
-      <origin xyz="0 0 0" rpy="0 0 0" />
-      <inertia ixx="0.0002" ixy="0" ixz="0" iyy="0.0002" iyz="0" izz="0.0002" />
-    </inertial>
-  </link>
-  <joint name="gps_joint" type="fixed">
-    <parent link="base_link" />
-    <child link="gps_link" />
-    <origin xyz="0 0 0.30" rpy="0 0 0" />
-  </joint>
   <!-- Camera -->
   <joint name="camera_joint" type="fixed">
@@ -229,10 +186,4 @@
   <xacro:property name="camera_size" value="0.05" /> <!-- Size of square 'camera' box -->
   <link name="camera_link">
-    <!--  <collision>
-      <geometry>
-          <box size=".1 .3 .1"/>
-      </geometry>
-      <contact_coefficients mu="0" kp="1000.0" kd="1.0"/>
-  </collision>-->
     <visual>
       <geometry>
@@ -249,32 +200,4 @@
     </inertial>
   </link>
-  <!-- LaserScan 230309 -->
-  <!-- <joint name="hokuyo_joint" type="fixed">
-    <axis xyz="0 1 0" />
-    <origin xyz="0 0 0.20" rpy="0 0 0"/>
-    <parent link="base_link"/>
-    <child link="hokuyo_link"/>
-  </joint> -->
-  <!-- <link name="hokuyo_link">
-    <collision>
-      <origin xyz="0 0 0" rpy="0 0 0"/>
-      <geometry>
-    <box size="0.1 0.1 0.1"/>
-      </geometry>
-    </collision>
-      <visual>
-    <geometry>
-      <cylinder radius="0.05" length="0.05"/>
-    </geometry>
-    <material name="blue">
-      <color rgba="1 1 1 0.5"/>
-    </material>
-  </visual>
-    <inertial>
-      <mass value="1e-5" />
-      <origin xyz="0 0 0" rpy="0 0 0"/>
-      <inertia ixx="1e-6" ixy="0" ixz="0" iyy="1e-6" iyz="0" izz="1e-6" />
-    </inertial>
-  </link> -->
   <!-- camera -->
   <gazebo reference="camera_link">
@@ -327,16 +250,5 @@
     </sensor>
   </gazebo>
-  <!-- <gazebo>
-    <plugin name="imu_plugin" filename="libgazebo_ros_imu.so">
-      <alwaysOn>true</alwaysOn>
-      <bodyName>imu_link</bodyName>
-      <topicName>imu</topicName>
-      <frameId>imu</frameId>
-      <serviceName>imu_service</serviceName>
-      <gaussianNoise>0.0</gaussianNoise>
-      <updateRate>100.0</updateRate>
-      <initialOrientationAsReference>false</initialOrientationAsReference>
-    </plugin>
-    </gazebo> -->
+  <!-- imu addon 230406chson -->
   <gazebo reference="imu_link">
     <gravity>true</gravity>
@@ -358,6 +270,19 @@
       <pose>0 0 0 0 0 0</pose>
     </sensor>
+    <!-- <sensor name="my_gps" type="gps"> -->
+  <!-- ensure the sensor is active (required) -->
+  <!-- <always_on>true</always_on> -->
+  <!-- <update_rate>30</update_rate> -->
+  <!-- <plugin name="my_gps_plugin" filename="libgazebo_ros_gps_sensor.so"> -->
+    <!-- <ros> -->
+      <!-- publish to /gps/data -->
+      <!-- <namespace>/gps</namespace> -->
+      <!-- <remapping>~/out:=data</remapping> -->
+    <!-- </ros> -->
+  <!-- </plugin> -->
+<!-- </sensor> -->
   </gazebo>
-  <!-- <gazebo>
+  <!-- gps addon 0406chson -->
+  <!-- <gazebo reference="gps_link">
     <plugin name="gps_controller" filename="libhector_gazebo_ros_gps.so">
       <alwayson>true</alwayson>
@@ -375,42 +300,3 @@
     </plugin>
   </gazebo> -->
-  <!-- <gazebo>
-    <gazebo reference="hokuyo_link">
-      <sensor type="ray" name="head_hokuyo_sensor">
-        <pose>0 0 0 0 0 0</pose>
-        <visualize>true</visualize>
-        <update_rate>40</update_rate>
-        <ray>
-          <scan>
-            <horizontal>
-              <samples>720</samples>
-              <resolution>1</resolution>
-              <min_angle>-1.570796</min_angle>
-              <min_angle>-150</min_angle>
-              <max_angle>1.570796</max_angle>
-              <max_angle>150</max_angle>
-            </horizontal>
-          </scan>
-          <range>
-            <min>0.10</min>
-            <max>300.0</max>
-            <resolution>0.01</resolution>
-          </range>
-          <noise>
-            <type>gaussian</type>
-            Noise parameters based on published spec for Hokuyo laser
-               achieving "+-30mm" accuracy at range < 10m.  A mean of 0.0m and
-               stddev of 0.01m will put 99.7% of samples within 0.03m of the true
-               reading.
-            <mean>0.0</mean>
-            <stddev>0.01</stddev>
-          </noise>
-        </ray>
-        <plugin name="gazebo_ros_head_hokuyo_controller" filename="libgazebo_ros_laser.so">
-          <topicName>/scan</topicName>
-          <frameName>hokuyo_link</frameName>
-        </plugin>
-      </sensor>
-    </gazebo>
-  </gazebo> -->
 </robot>
